Commit message: MUIN First commit

File: urdf/mid360.xacro (robot description, xacro)
@@ -23,6 +23,7 @@
 <xacro:box_inertia m="${length}" w="${width}" d="${length}" h="${height}"/>
   <visual>
+  	<origin xyz="0.025 -0.0265 -0.025" rpy="${pi/2} 0 ${pi}"/>
         <geometry>
-            <box size="${length} ${width} ${height}"/>
+            <mesh filename="$(find ros2_livox_simulation)/meshes/mid360.stl" scale="0.0008 0.0008 0.0008"/>
         </geometry>
   </visual>
